Commit message: Added configurations for Jackal robot to speed up simulation.

File: src/jackal/jackal_description/urdf/accessories.urdf.xacro (robot description, xacro)
@@ -10,10 +10,12 @@
   -->
   <!-- Implement the Velodyne-32 Sensor. -->
-  <xacro:include filename="$(find jackal_description)/urdf/accessories/HDL-32E.urdf.xacro"/>
-  <xacro:arg name="gpu" default="false"/>
-  <xacro:property name="gpu" value="$(arg gpu)" />
-  <HDL-32E parent="base_link" name="velodyne2" topic="/velodyne_points2" hz="10" samples="110" gpu="${gpu}">
-    <origin xyz="0 0 0.15" rpy="0 0 0" />
-  </HDL-32E>
+  <xacro:if value="$(optenv JACKAL_VELODYNE 0)">
+    <xacro:include filename="$(find jackal_description)/urdf/accessories/HDL-32E.urdf.xacro"/>
+    <xacro:arg name="gpu" default="false"/>
+    <xacro:property name="gpu" value="$(arg gpu)" />
+    <HDL-32E parent="base_link" name="velodyne2" topic="/velodyne_points2" hz="10" samples="110" gpu="${gpu}">
+      <origin xyz="0 0 0.15" rpy="0 0 0" />
+    </HDL-32E>
+  </xacro:if>
   <!-- Macros to generate standoffs for offset payload mounting. -->
   <xacro:include filename="$(find jackal_description)/urdf/accessories/standoffs.urdf.xacro" />

Commit message: Improved trajectory planner. Simplified file structure.

File: src/jackal/jackal_description/urdf/accessories.urdf.xacro (robot description, xacro)
@@ -15,4 +15,12 @@
     <xacro:property name="gpu" value="$(arg gpu)" />
     <HDL-32E parent="base_link" name="velodyne2" topic="/velodyne_points2" hz="20" samples="110" gpu="${gpu}">
+      <origin xyz="0 0 0.15" rpy="0 0 0" />
+    </HDL-32E>
+  </xacro:if>
+  <xacro:if value="$(optenv JACKAL_VELODYNE_HD 0)">
+    <xacro:include filename="$(find jackal_description)/urdf/accessories/HDL-32E.urdf.xacro"/>
+    <xacro:arg name="gpu" default="false"/>
+    <xacro:property name="gpu" value="$(arg gpu)" />
+    <HDL-32E parent="base_link" name="velodyne2" topic="/velodyne_points2" hz="20" samples="220" gpu="${gpu}">
       <origin xyz="0 0 0.15" rpy="0 0 0" />
     </HDL-32E>

Commit message: Updated Velodyne model link.

File: src/jackal/jackal_description/urdf/accessories.urdf.xacro (robot description, xacro)
@@ -11,18 +11,14 @@
   <!-- Implement the Velodyne-32 Sensor. -->
   <xacro:if value="$(optenv JACKAL_VELODYNE 0)">
-    <xacro:include filename="$(find jackal_description)/urdf/accessories/HDL-32E.urdf.xacro"/>
-    <xacro:arg name="gpu" default="false"/>
-    <xacro:property name="gpu" value="$(arg gpu)" />
-    <HDL-32E parent="base_link" name="velodyne2" topic="/velodyne_points2" hz="20" samples="110" gpu="${gpu}">
-      <origin xyz="0 0 0.15" rpy="0 0 0" />
-    </HDL-32E>
+    <xacro:include filename="$(find jackal_description)/urdf/accessories/HDL-32E.urdf.xacro" />
+    <xacro:HDL-32E parent="$(optenv JACKAL_LASER_MOUNT front)_mount" name="velodyne2" topic="/velodyne_points2" hz="10" samples="110" >
+      <origin xyz="0 0 0" rpy="0 0 0" />
+    </xacro:HDL-32E>
   </xacro:if>
   <xacro:if value="$(optenv JACKAL_VELODYNE_HD 0)">
-    <xacro:include filename="$(find jackal_description)/urdf/accessories/HDL-32E.urdf.xacro"/>
-    <xacro:arg name="gpu" default="false"/>
-    <xacro:property name="gpu" value="$(arg gpu)" />
-    <HDL-32E parent="base_link" name="velodyne2" topic="/velodyne_points2" hz="20" samples="220" gpu="${gpu}">
-      <origin xyz="0 0 0.15" rpy="0 0 0" />
-    </HDL-32E>
+    <xacro:include filename="$(find jackal_description)/urdf/accessories/HDL-32E.urdf.xacro" />
+    <xacro:HDL-32E parent="$(optenv JACKAL_LASER_MOUNT front)_mount" name="velodyne2" topic="/velodyne_points2" hz="20" samples="220" >
+      <origin xyz="0 0 0" rpy="0 0 0" />
+    </xacro:HDL-32E>
   </xacro:if>
   <!-- Macros to generate standoffs for offset payload mounting. -->

File: src/jackal/jackal_description/urdf/jackal.urdf.xacro (robot description, xacro)
@@ -184,5 +184,5 @@
     <inertial>
       <mass value="0.001"/>
-      <origin xyz="0 0 0" rpy="0 0 0"/>
+      <origin xyz="${orig_xyz}" rpy="0 0 0"/>
       <inertia ixx="${dummy_inertia}" ixy="0.0" ixz="0.0" iyy="${dummy_inertia}" iyz="0.0" izz="${dummy_inertia}"/>
     </inertial>
@@ -198,5 +198,5 @@
         <cylinder radius="0.026" length="0.016" />
       </geometry>
-      <origin xyz="0 0 0.008" />
+      <origin xyz="${orig_x} ${orig_y} 0.008" />
       <material name="black" />
     </visual>
