Commit message: Added Jackal sensor configurations.

File: src/jackal/jackal_description/urdf/jackal.urdf.xacro (robot description, xacro)
@@ -1,4 +1,5 @@
 <?xml version="1.0"?>
 <robot name="jackal" xmlns:xacro="http://www.ros.org/wiki/xacro">
+  <!-- Attempting to shift the robot starting position -->
   <xacro:property name="orig_x" value="0" />
   <xacro:property name="orig_y" value="0" />
@@ -84,4 +85,13 @@
     <origin xyz="${-wheelbase/2} ${-track/2} ${wheel_vertical_offset}" rpy="0 0 0" />
   </xacro:wheel>
+ <!--
+  <link name="world" />
+   <link name="link0" />
+   <joint name="world_joint" type="fixed">
+     <parent link="world" />
+     <child link="link0" />
+     <origin xyz="0 0 0" rpy="0 0 0"/>
+     <axis xyz="0 0 1"/>
+   </joint>-->
   <link name="base_link"></link>
   <joint name="base_link_joint" type="fixed">

Commit message: Updated pedestrian simulation rate.

File: src/jackal/jackal_description/urdf/jackal.urdf.xacro (robot description, xacro)
@@ -85,13 +85,4 @@
     <origin xyz="${-wheelbase/2} ${-track/2} ${wheel_vertical_offset}" rpy="0 0 0" />
   </xacro:wheel>
- <!--
-  <link name="world" />
-   <link name="link0" />
-   <joint name="world_joint" type="fixed">
-     <parent link="world" />
-     <child link="link0" />
-     <origin xyz="0 0 0" rpy="0 0 0"/>
-     <axis xyz="0 0 1"/>
-   </joint>-->
   <link name="base_link"></link>
   <joint name="base_link_joint" type="fixed">
